File: pcb/hardware.kicad_pcb (KiCad board)
At the start: 4 copper layers, 59 x 53 mm, 144 parts, among them J1 Micro_SD_Card_Det_Hirose_DM3AT, J2 USB_A, J3 USB_A, J5 Conn_02x10_Odd_Even, U1 AS4C512M16D3L-12BIN, U2 A33, U3 TPS62095RGTR, U4 TPS62095RGTR, U5 TPS62095RGTR, U6 TPS62095RGTR, U7 AP131-25, Y1 24Mhz, Y2 32.768khz

Commit message: Working on the board
Routing:
- net /gpio/SD_CLK: track 0.00 -> 11.3 mm, vias 0 -> 2
- net +3V3: track 5.28 -> 15.1 mm, vias 3 -> 10
- net /gpio/SD_DAT3: track 0.00 -> 7.77 mm
- net /gpio/SD_CMD: track 0.00 -> 7.09 mm
- net /gpio/SD_DAT2: track 0.00 -> 6.82 mm
- net +3V0: track 9.79 -> 12.4 mm
- net +1V1: vias 5 -> 11
- added copper zone on In1.Cu, net +1V1
- added copper zone on In1.Cu, net +3V3
Changed lines of the file:
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@@
     (thickness 1.6)
     (drawings 14)
-    (tracks 16494)
+    (tracks 16539)
     (zones 0)
     (modules 144)
@@
     (0 F.Cu signal)
     (1 In1.Cu signal)
-    (2 In2.Cu signal)
+    (2 In2.Cu signal hide)
     (31 B.Cu signal)
     (32 B.Adhes user hide)
@@
     (34 B.Paste user hide)
     (35 F.Paste user hide)
-    (36 B.SilkS user)
-    (37 F.SilkS user)
+    (36 B.SilkS user hide)
+    (37 F.SilkS user hide)
     (38 B.Mask user hide)
     (39 F.Mask user hide)
@@
   )
   (setup
-    (last_trace_width 0.15)
+    (last_trace_width 0.1)
     (user_trace_width 0.1)
+    (user_trace_width 0.5)
+    (user_trace_width 1)
     (trace_clearance 0.15)
     (zone_clearance 0.127)
@@
     (via_min_drill 0.2)
     (user_via 0.4 0.2)
+    (user_via 0.4 0.3)
+    (user_via 1 0.5)
     (uvia_size 0.4)
     (uvia_drill 0.2)
@@
   (gr_line (start 154 137) (end 154 84) (layer Edge.Cuts) (width 0.05))
   (gr_line (start 95 137) (end 154 137) (layer Edge.Cuts) (width 0.05))
+  (via (at 141.224 129.794) (size 0.4) (drill 0.2) (layers F.Cu B.Cu) (net 193))
+  (via (at 141.224 130.3274) (size 0.4) (drill 0.2) (layers F.Cu B.Cu) (net 193))
+  (via (at 140.716 130.3274) (size 0.4) (drill 0.2) (layers F.Cu B.Cu) (net 193))
+  (via (at 140.716 129.794) (size 0.4) (drill 0.2) (layers F.Cu B.Cu) (net 193))
+  (via (at 140.716 129.2606) (size 0.4) (drill 0.2) (layers F.Cu B.Cu) (net 193))
   (via (at 140.589 115.2652) (size 0.4) (drill 0.2) (layers F.Cu B.Cu) (net 168))
   (via (at 140.589 115.7732) (size 0.4) (drill 0.2) (layers F.Cu B.Cu) (net 168))
@@
   (segment (start 138.178 116.33) (end 137.7442 116.7638) (width 0.15) (layer F.Cu) (net 168))
   (segment (start 139.3444 116.33) (end 138.178 116.33) (width 0.15) (layer F.Cu) (net 168))
+  (via (at 141.224 129.2606) (size 0.4) (drill 0.2) (layers F.Cu B.Cu) (net 193))
   (via (at 118.364 108.5596) (size 0.4) (drill 0.2) (layers F.Cu B.Cu) (net 170))
   (segment (start 118.7572 108.1664) (end 118.364 108.5596) (width 0.1) (layer F.Cu) (net 170))
@@
   (segment (start 113.1572 106.566) (end 112.3572 106.566) (width 0.15) (layer F.Cu) (net 194))
   (segment (start 111.5572 107.366) (end 111.79332 107.12988) (width 0.15) (layer F.Cu) (net 194))
-  (segment (start 111.5572 108.166) (end 111.5572 107.366) (width 0.15) (layer F.Cu) (net 194))
   (segment (start 111.79332 107.12988) (end 112.3572 106.566) (width 0.15) (layer F.Cu) (net 194))
   (via (at 111.79332 107.12988) (size 0.4) (drill 0.2) (layers F.Cu B.Cu) (net 194))
@@
   (segment (start 108.762199 106.970999) (end 107.326201 106.970999) (width 0.15) (layer F.Cu) (net 194))
   (segment (start 109.1572 107.366) (end 108.762199 106.970999) (width 0.15) (layer F.Cu) (net 194))
+  (segment (start 111.545601 107.761001) (end 111.5572 107.7726) (width 0.15) (layer F.Cu) (net 194))
+  (segment (start 109.552201 107.761001) (end 111.545601 107.761001) (width 0.15) (layer F.Cu) (net 194))
+  (segment (start 109.1572 107.366) (end 109.552201 107.761001) (width 0.15) (layer F.Cu) (net 194))
+  (segment (start 111.5572 107.7726) (end 111.5572 107.366) (width 0.15) (layer F.Cu) (net 194))
+  (segment (start 111.5572 108.166) (end 111.5572 107.7726) (width 0.15) (layer F.Cu) (net 194))
   (via (at 116.7638 105.3592) (size 0.4) (drill 0.2) (layers F.Cu B.Cu) (net 195))
   (segment (start 117.1572 105.7526) (end 116.7638 105.3592) (width 0.15) (layer F.Cu) (net 195))
@@
   (segment (start 110.5053 112.1918) (end 110.49 112.1765) (width 0.15) (layer B.Cu) (net 195))
   (segment (start 112.3188 112.1918) (end 110.5053 112.1918) (width 0.15) (layer B.Cu) (net 195))
+  (via (at 150.622 121.3485) (size 0.4) (drill 0.2) (layers F.Cu B.Cu) (net 195))
+  (via (at 150.114 121.3485) (size 0.4) (drill 0.2) (layers F.Cu B.Cu) (net 195))
+  (via (at 149.606 121.3485) (size 0.4) (drill 0.2) (layers F.Cu B.Cu) (net 195))
+  (via (at 149.098 121.3485) (size 0.4) (drill 0.2) (layers F.Cu B.Cu) (net 195))
+  (via (at 148.59 121.3485) (size 0.4) (drill 0.2) (layers F.Cu B.Cu) (net 195))
+  (via (at 105.283 104.9655) (size 0.4) (drill 0.2) (layers F.Cu B.Cu) (net 195))
+  (segment (start 105.4608 105.1433) (end 105.283 104.9655) (width 0.15) (layer F.Cu) (net 195))
+  (segment (start 106.0811 105.1433) (end 105.4608 105.1433) (width 0.15) (layer F.Cu) (net 195))
+  (segment (start 105.283 104.9655) (end 107.188 104.9655) (width 1) (layer In1.Cu) (net 195))
+  (via (at 108.7628 104.5464) (size 0.4) (drill 0.2) (layers F.Cu B.Cu) (net 195))
+  (segment (start 108.839 104.4702) (end 108.7628 104.5464) (width 0.15) (layer B.Cu) (net 195))
+  (segment (start 109.5736 104.4702) (end 108.839 104.4702) (width 0.15) (layer B.Cu) (net 195))
+  (segment (start 108.7628 104.5464) (end 108.7628 106.4006) (width 0.15) (layer In1.Cu) (net 195))
+  (segment (start 108.7628 106.4006) (end 108.69295 106.47045) (width 0.15) (layer In1.Cu) (net 195))
+  (segment (start 108.69295 106.47045) (end 110.1725 107.95) (width 1) (layer In1.Cu) (net 195))
+  (segment (start 107.188 104.9655) (end 108.69295 106.47045) (width 1) (layer In1.Cu) (net 195))
   (segment (start 148.03374 112.0688) (end 148.9797 112.0688) (width 0.15) (layer F.Cu) (net 196))
   (via (at 148.9964 112.0521) (size 0.4) (drill 0.2) (layers F.Cu B.Cu) (net 196))
@@
   (segment (start 140.04982 125.6959) (end 140.04982 126.57198) (width 0.15) (layer F.Cu) (net 219))
   (segment (start 138.7348 126.871) (end 139.7508 126.871) (width 0.15) (layer F.Cu) (net 219))
+  (via (at 115.1636 113.3602) (size 0.4) (drill 0.2) (layers F.Cu B.Cu) (net 225))
+  (segment (start 115.5572 112.9666) (end 115.1636 113.3602) (width 0.1) (layer F.Cu) (net 225))
+  (segment (start 115.5572 112.966) (end 115.5572 112.9666) (width 0.1) (layer F.Cu) (net 225))
+  (segment (start 115.1636 113.3602) (end 115.1636 117.9576) (width 0.1) (layer B.Cu) (net 225))
+  (via (at 111.7092 121.412) (size 0.4) (drill 0.2) (layers F.Cu B.Cu) (net 225))
+  (segment (start 115.1636 117.9576) (end 111.7092 121.412) (width 0.1) (layer B.Cu) (net 225))
+  (segment (start 111.7092 120.1888) (end 111.6844 120.164) (width 0.1) (layer F.Cu) (net 225))
+  (segment (start 111.7092 121.412) (end 111.7092 120.1888) (width 0.1) (layer F.Cu) (net 225))
+  (segment (start 113.8844 119.953998) (end 113.8844 120.164) (width 0.1) (layer F.Cu) (net 226))
+  (segment (start 115.127201 118.711197) (end 113.8844 119.953998) (width 0.1) (layer F.Cu) (net 226))
+  (segment (start 115.127201 114.195999) (end 115.127201 118.711197) (width 0.1) (layer F.Cu) (net 226))
+  (segment (start 115.5572 113.766) (end 115.127201 114.195999) (width 0.1) (layer F.Cu) (net 226))
+  (segment (start 115.987199 118.951199) (end 114.9844 119.953998) (width 0.1) (layer F.Cu) (net 227))
+  (segment (start 114.9844 119.953998) (end 114.9844 120.164) (width 0.1) (layer F.Cu) (net 227))
+  (segment (start 115.987199 113.336001) (end 115.987199 118.951199) (width 0.1) (layer F.Cu) (net 227))
+  (segment (start 116.3572 112.966) (end 115.987199 113.336001) (width 0.1) (layer F.Cu) (net 227))
+  (segment (start 116.727201 114.136001) (end 116.727201 119.521199) (width 0.1) (layer F.Cu) (net 228))
+  (segment (start 116.727201 119.521199) (end 116.0844 120.164) (width 0.1) (layer F.Cu) (net 228))
+  (segment (start 116.3572 113.766) (end 116.727201 114.136001) (width 0.1) (layer F.Cu) (net 228))
   (segment (start 107.61421 111.12799) (end 107.1092 111.633) (width 0.15) (layer F.Cu) (net 230))
   (segment (start 107.61421 110.50899) (end 107.61421 111.12799) (width 0.15) (layer F.Cu) (net 230))
@@
       )
     )
+  )
+  (zone (net 195) (net_name +3V3) (layer F.Cu) (hatch edge 0.508)
+    (priority 1)
+    (connect_pads yes (clearance 0.127))
+    (min_thickness 0.254)
+    (fill yes (arc_segments 32) (thermal_gap 0.508) (thermal_bridge_width 0.508))
+    (polygon
+      (pts
+        (xy 150.876 121.666) (xy 147.574 121.666) (xy 147.574 119.888) (xy 148.7805 119.888) (xy 149.479 118.872)
+        (xy 150.876 118.872)
+      )
+    )
+  )
+  (zone (net 195) (net_name +3V3) (layer In1.Cu) (hatch edge 0.508)
+    (priority 1)
+    (connect_pads yes (clearance 0.127))
+    (min_thickness 0.254)
+    (fill yes (arc_segments 32) (thermal_gap 0.508) (thermal_bridge_width 0.508))
+    (polygon
+      (pts
+        (xy 113.0046 113.4745) (xy 117.8814 120.1674) (xy 117.856 132.5118) (xy 142.0495 132.461) (xy 145.415 129.286)
+        (xy 146.6215 121.0945) (xy 152.7175 121.0945) (xy 152.7175 136.5885) (xy 128.27 136.525) (xy 124.0155 135.0645)
+        (xy 109.7915 135.0645) (xy 109.7915 107.315) (xy 112.3315 107.315) (xy 112.3315 108.1405) (xy 111.125 108.1405)
+        (xy 111.125 109.855) (xy 113.0046 109.855)
+      )
+    )
+  )
+  (zone (net 193) (net_name +1V1) (layer F.Cu) (hatch edge 0.508)
+    (priority 1)
+    (connect_pads yes (clearance 0.127))
+    (min_thickness 0.254)
+    (fill yes (arc_segments 32) (thermal_gap 0.508) (thermal_bridge_width 0.508))
+    (polygon
+      (pts
+        (xy 141.6558 132.2578) (xy 139.6492 132.2578) (xy 139.6492 130.683) (xy 139.0904 130.683) (xy 139.0904 128.9304)
+        (xy 141.6558 128.9304)
+      )
+    )
+  )
+  (zone (net 193) (net_name +1V1) (layer In1.Cu) (hatch edge 0.508)
+    (priority 1)
+    (connect_pads yes (clearance 0.127))
+    (min_thickness 0.254)
+    (fill yes (arc_segments 32) (thermal_gap 0.508) (thermal_bridge_width 0.508))
+    (polygon
+      (pts
+        (xy 117.1702 106.1212) (xy 117.1702 110.1344) (xy 118.0338 110.1344) (xy 118.0338 112.9792) (xy 126.3142 120.1928)
+        (xy 126.3142 128.9558) (xy 142.0368 128.9558) (xy 142.0368 131.3942) (xy 122.6058 131.4196) (xy 122.6566 120.4214)
+        (xy 113.9952 113.2586) (xy 113.9952 107.5944) (xy 111.4806 106.5784) (xy 111.4806 104.6988) (xy 115.7732 104.6988)
+      )
+    )
