File: pcb/gpio.sch (KiCad schematic (older format))
At the start: 31 parts, among them J1 Micro_SD_Card_Det_Hirose_DM3AT, J2 USB_A, J3 USB_A, J4 Conn_01x03_Male, U2 A33, Y1 24Mhz, Y2 32.768khz

Commit message: Working on silkscreen/placement
Parts:
- removed J4: Conn_01x03_Male, symbol Connector:Conn_01x03_Male
- added J5: Conn_02x10_Odd_Even, Connector_PinHeader_2.54mm:PinHeader_2x10_P2.54mm_Vertical, symbol Connector_Generic:Conn_02x10_Odd_Even
Connections:
- net UART0_RX: now also J5.3 (Pin_3)
- net UART0_TX: now also J5.1 (Pin_1)
Changed lines of the file:
@@
 Text Label 1600 1050 2    50   ~ 0
 UART0_RX
+Wire Wire Line
+	1600 950  1750 950
+Wire Wire Line
+	1600 1050 1750 1050
 $Comp
-L Connector:Conn_01x03_Male J4
-U 1 1 60978C13
-P 750 1050
-F 0 "J4" H 850 1400 50  0000 C CNN
-F 1 "Conn_01x03_Male" H 850 1300 50  0000 C CNN
-F 2 "" H 750 1050 50  0001 C CNN
-F 3 "~" H 750 1050 50  0001 C CNN
-	1    750  1050
+L Connector_Generic:Conn_02x10_Odd_Even J5
+U 1 1 608A0623
+P 4500 5550
+F 0 "J5" H 4550 6167 50  0000 C CNN
+F 1 "Conn_02x10_Odd_Even" H 4550 6076 50  0000 C CNN
+F 2 "Connector_PinHeader_2.54mm:PinHeader_2x10_P2.54mm_Vertical" H 4500 5550 50  0001 C CNN
+F 3 "~" H 4500 5550 50  0001 C CNN
+	1    4500 5550
 	1    0    0    -1
 $EndComp
+Text Label 4050 5150 2    50   ~ 0
+UART0_TX
+Text Label 4050 5250 2    50   ~ 0
+UART0_RX
 Wire Wire Line
-	950  950  1750 950
+	4050 5150 4300 5150
 Wire Wire Line
-	950  1050 1750 1050
-Wire Wire Line
-	950  1150 1000 1150
-Wire Wire Line
-	1000 1150 1000 1200
-$Comp
-L power:GND #PWR?
-U 1 1 609DD2CB
-P 1000 1200
-AR Path="/60536DA4/609DD2CB" Ref="#PWR?"  Part="1"
-AR Path="/609DD2CB" Ref="#PWR?"  Part="1"
-AR Path="/60A30BFF/609DD2CB" Ref="#PWR?"  Part="1"
-AR Path="/6063BE69/609DD2CB" Ref="#PWR084"  Part="1"
-F 0 "#PWR084" H 1000 950 50  0001 C CNN
-F 1 "GND" V 1005 1072 50  0001 R CNN
-F 2 "" H 1000 1200 50  0001 C CNN
-F 3 "" H 1000 1200 50  0001 C CNN
-	1    1000 1200
-	1    0    0    -1
-$EndComp
+	4300 5250 4050 5250
 $EndSCHEMATC

Commit message: Still working on the routing.
Connections:
- net +5V: now also J5.2 (Pin_2)
- net GND: now also J5.1 (Pin_1)
- net UART0_RX: now also J5.18 (Pin_18); no longer J5.3 (Pin_3)
- net UART0_TX: now also J5.20 (Pin_20); no longer J5.1 (Pin_1)
Changed lines of the file:
@@
 	1    0    0    -1
 $EndComp
-Text Label 4050 5150 2    50   ~ 0
+Text Label 5050 6050 0    50   ~ 0
 UART0_TX
-Text Label 4050 5250 2    50   ~ 0
+Text Label 5050 5950 0    50   ~ 0
 UART0_RX
 Wire Wire Line
-	4050 5150 4300 5150
+	5050 6050 4800 6050
 Wire Wire Line
-	4300 5250 4050 5250
+	4800 5950 5050 5950
+$Comp
+L power:GND #PWR?
+U 1 1 609FA802
+P 4150 5150
+AR Path="/60536DA4/609FA802" Ref="#PWR?"  Part="1"
+AR Path="/609FA802" Ref="#PWR?"  Part="1"
+AR Path="/60A30BFF/609FA802" Ref="#PWR?"  Part="1"
+AR Path="/6063BE69/609FA802" Ref="#PWR0109"  Part="1"
+F 0 "#PWR0109" H 4150 4900 50  0001 C CNN
+F 1 "GND" V 4155 5022 50  0001 R CNN
+F 2 "" H 4150 5150 50  0001 C CNN
+F 3 "" H 4150 5150 50  0001 C CNN
+	1    4150 5150
+	0    1    1    0
+$EndComp
+Wire Wire Line
+	4150 5150 4300 5150
+Wire Wire Line
+	4800 5150 5050 5150
+Wire Wire Line
+	5050 5150 5050 5000
+$Comp
+L power:+5V #PWR?
+U 1 1 60A0F4D1
+P 5050 5000
+AR Path="/60A30BFF/60A0F4D1" Ref="#PWR?"  Part="1"
+AR Path="/6063BE69/60A0F4D1" Ref="#PWR0110"  Part="1"
+F 0 "#PWR0110" H 5050 4850 50  0001 C CNN
+F 1 "+5V" H 5065 5173 50  0000 C CNN
+F 2 "" H 5050 5000 50  0001 C CNN
+F 3 "" H 5050 5000 50  0001 C CNN
+	1    5050 5000
+	1    0    0    -1
+$EndComp
 $EndSCHEMATC

Commit message: Routing
Connections:
- net GND: now also J5.11 (Pin_11), J5.13 (Pin_13)
- net UART0_RX: now also J5.14 (Pin_14); no longer J5.18 (Pin_18)
- net UART0_TX: now also J5.12 (Pin_12); no longer J5.20 (Pin_20)
- net PG8: now reaches U2.A16 (PG8)
- net PG8: now also J5.20 (Pin_20)
- net PG6: now reaches U2.A17 (PG6)
- net PG6: now also J5.19 (Pin_19)
- net PG9: now reaches U2.B16 (PG9)
- net PG9: now also J5.18 (Pin_18)
- net PG7: now reaches U2.B17 (PG7)
- net PG7: now also J5.17 (Pin_17)
- net PG11: now reaches U2.C16 (PG11)
- net PG11: now also J5.16 (Pin_16)
- net PG10: now reaches U2.C17 (PG10)
- net PG10: now also J5.15 (Pin_15)
Changed lines of the file:
@@
 	1    0    0    -1
 $EndComp
-Text Label 5050 6050 0    50   ~ 0
+Text Label 4950 5650 0    50   ~ 0
 UART0_TX
-Text Label 5050 5950 0    50   ~ 0
+Text Label 4950 5750 0    50   ~ 0
 UART0_RX
 Wire Wire Line
-	5050 6050 4800 6050
+	4950 5750 4800 5750
 Wire Wire Line
-	4800 5950 5050 5950
+	4800 5650 4950 5650
 $Comp
 L power:GND #PWR?
@@
 	1    0    0    -1
 $EndComp
+Wire Wire Line
+	2650 4150 2800 4150
+Text Label 2800 4150 0    50   ~ 0
+PG6
+Wire Wire Line
+	2650 4350 2800 4350
+Text Label 2800 4350 0    50   ~ 0
+PG8
+Text Label 4100 6050 0    50   ~ 0
+PG6
+Wire Wire Line
+	4100 6050 4300 6050
+Wire Wire Line
+	4800 6050 4950 6050
+Text Label 4950 6050 0    50   ~ 0
+PG8
+Wire Wire Line
+	2650 4250 2800 4250
+Text Label 2800 4250 0    50   ~ 0
+PG7
+Text Label 4100 5950 0    50   ~ 0
+PG7
+Wire Wire Line
+	4100 5950 4300 5950
+Wire Wire Line
+	2650 4450 2800 4450
+Text Label 2800 4450 0    50   ~ 0
+PG9
+Wire Wire Line
+	4800 5950 4950 5950
+Text Label 4950 5950 0    50   ~ 0
+PG9
+Wire Wire Line
+	2650 4550 2800 4550
+Text Label 2800 4550 0    50   ~ 0
+PG10
+Wire Wire Line
+	2650 4650 2800 4650
+Text Label 2800 4650 0    50   ~ 0
+PG11
+Text Label 4100 5850 0    50   ~ 0
+PG10
+Wire Wire Line
+	4800 5850 4950 5850
+Text Label 4950 5850 0    50   ~ 0
+PG11
+Wire Wire Line
+	4300 5850 4100 5850
+$Comp
+L power:GND #PWR?
+U 1 1 609F201D
+P 4150 5750
+AR Path="/60536DA4/609F201D" Ref="#PWR?"  Part="1"
+AR Path="/609F201D" Ref="#PWR?"  Part="1"
+AR Path="/60A30BFF/609F201D" Ref="#PWR?"  Part="1"
+AR Path="/6063BE69/609F201D" Ref="#PWR?"  Part="1"
+F 0 "#PWR?" H 4150 5500 50  0001 C CNN
+F 1 "GND" V 4155 5622 50  0001 R CNN
+F 2 "" H 4150 5750 50  0001 C CNN
+F 3 "" H 4150 5750 50  0001 C CNN
+	1    4150 5750
+	0    1    1    0
+$EndComp
+Wire Wire Line
+	4150 5750 4300 5750
+$Comp
+L power:GND #PWR?
+U 1 1 609FB83F
+P 4150 5650
+AR Path="/60536DA4/609FB83F" Ref="#PWR?"  Part="1"
+AR Path="/609FB83F" Ref="#PWR?"  Part="1"
+AR Path="/60A30BFF/609FB83F" Ref="#PWR?"  Part="1"
+AR Path="/6063BE69/609FB83F" Ref="#PWR?"  Part="1"
+F 0 "#PWR?" H 4150 5400 50  0001 C CNN
+F 1 "GND" V 4155 5522 50  0001 R CNN
+F 2 "" H 4150 5650 50  0001 C CNN
+F 3 "" H 4150 5650 50  0001 C CNN
+	1    4150 5650
+	0    1    1    0
+$EndComp
+Wire Wire Line
+	4150 5650 4300 5650
 $EndSCHEMATC

Commit message: Moving stuff around
Connections:
- net +3V3: now also J5.8 (Pin_8)
- net USB-DM0: now reaches J2.2 (D-), U2.T16 (USB-DM0)
- net USB-DP0: now reaches J2.3 (D+), U2.T17 (USB-DP0)
- net USB-DM1: now reaches J3.2 (D-), U2.U16 (USB-DM1)
- net USB-DP1: now reaches J3.3 (D+), U2.U17 (USB-DP1)
- net +1V1: now reaches J5.5 (Pin_5)
- net +1V35: now reaches J5.6 (Pin_6)
- net +3V0: now reaches J5.7 (Pin_7)
Changed lines of the file:
@@
 AR Path="/609F201D" Ref="#PWR?"  Part="1"
 AR Path="/60A30BFF/609F201D" Ref="#PWR?"  Part="1"
-AR Path="/6063BE69/609F201D" Ref="#PWR?"  Part="1"
-F 0 "#PWR?" H 4150 5500 50  0001 C CNN
+AR Path="/6063BE69/609F201D" Ref="#PWR0111"  Part="1"
+F 0 "#PWR0111" H 4150 5500 50  0001 C CNN
 F 1 "GND" V 4155 5622 50  0001 R CNN
 F 2 "" H 4150 5750 50  0001 C CNN
@@
 AR Path="/609FB83F" Ref="#PWR?"  Part="1"
 AR Path="/60A30BFF/609FB83F" Ref="#PWR?"  Part="1"
-AR Path="/6063BE69/609FB83F" Ref="#PWR?"  Part="1"
-F 0 "#PWR?" H 4150 5400 50  0001 C CNN
+AR Path="/6063BE69/609FB83F" Ref="#PWR0112"  Part="1"
+F 0 "#PWR0112" H 4150 5400 50  0001 C CNN
 F 1 "GND" V 4155 5522 50  0001 R CNN
 F 2 "" H 4150 5650 50  0001 C CNN
@@
 Wire Wire Line
 	4150 5650 4300 5650
+$Comp
+L power:+3V0 #PWR?
+U 1 1 60948FA9
+P 3600 5150
+AR Path="/60A30BFF/60948FA9" Ref="#PWR?"  Part="1"
+AR Path="/60948FA9" Ref="#PWR?"  Part="1"
+AR Path="/6063BE69/60948FA9" Ref="#PWR0113"  Part="1"
+F 0 "#PWR0113" H 3600 5000 50  0001 C CNN
+F 1 "+3V0" H 3615 5323 50  0000 C CNN
+F 2 "" H 3600 5150 50  0001 C CNN
+F 3 "" H 3600 5150 50  0001 C CNN
+	1    3600 5150
+	1    0    0    -1
+$EndComp
+$Comp
+L power:+3V3 #PWR?
+U 1 1 60948FB6
+P 5650 5100
+AR Path="/60A30BFF/60948FB6" Ref="#PWR?"  Part="1"
+AR Path="/60948FB6" Ref="#PWR?"  Part="1"
+AR Path="/6063BE69/60948FB6" Ref="#PWR0114"  Part="1"
+F 0 "#PWR0114" H 5650 4950 50  0001 C CNN
+F 1 "+3V3" H 5665 5273 50  0000 C CNN
+F 2 "" H 5650 5100 50  0001 C CNN
+F 3 "" H 5650 5100 50  0001 C CNN
+	1    5650 5100
+	1    0    0    -1
+$EndComp
+Wire Wire Line
+	4800 5450 5650 5450
+Wire Wire Line
+	5650 5450 5650 5100
+Wire Wire Line
+	4300 5450 3600 5450
+Wire Wire Line
+	3600 5450 3600 5150
+$Comp
+L power:+1V35 #PWR?
+U 1 1 609B2DEF
+P 5400 5100
+AR Path="/60536DA4/609B2DEF" Ref="#PWR?"  Part="1"
+AR Path="/60A30BFF/609B2DEF" Ref="#PWR?"  Part="1"
+AR Path="/609B2DEF" Ref="#PWR?"  Part="1"
+AR Path="/6063BE69/609B2DEF" Ref="#PWR0115"  Part="1"
+F 0 "#PWR0115" H 5400 4950 50  0001 C CNN
+F 1 "+1V35" H 5415 5273 50  0000 C CNN
+F 2 "" H 5400 5100 50  0001 C CNN
+F 3 "" H 5400 5100 50  0001 C CNN
+	1    5400 5100
+	1    0    0    -1
+$EndComp
+Wire Wire Line
+	5400 5100 5400 5350
+Wire Wire Line
+	5400 5350 4800 5350
+$Comp
+L power:+1V1 #PWR?
+U 1 1 60A095D8
+P 3800 5150
+AR Path="/60A30BFF/60A095D8" Ref="#PWR?"  Part="1"
+AR Path="/60A095D8" Ref="#PWR?"  Part="1"
+AR Path="/6063BE69/60A095D8" Ref="#PWR0116"  Part="1"
+F 0 "#PWR0116" H 3800 5000 50  0001 C CNN
+F 1 "+1V1" H 3815 5323 50  0000 C CNN
+F 2 "" H 3800 5150 50  0001 C CNN
+F 3 "" H 3800 5150 50  0001 C CNN
+	1    3800 5150
+	1    0    0    -1
+$EndComp
+Wire Wire Line
+	3800 5150 3800 5350
+Wire Wire Line
+	3800 5350 4300 5350
+Text Label 6600 2850 0    50   ~ 0
+USB-DP0
+Text Label 6600 2950 0    50   ~ 0
+USB-DM0
+Text Label 6600 3600 0    50   ~ 0
+USB-DP1
+Text Label 6600 3700 0    50   ~ 0
+USB-DM1
 $EndSCHEMATC
