File: electronics/pcb/a33_power.sch (KiCad schematic (older format))
At the start: 56 parts, among them U3 TPS62095RGTR, U4 TPS62095RGTR, U5 TPS62095RGTR, U6 TPS62095RGTR, U7 AP131-25

Commit message: DRC + BOM script
Parts:
- U3, U4, U5, U6: MPN (none) -> TPS62095RGTR
- U7: MPN (none) -> AP131-25
Changed lines of the file:
@@
 F 2 "TI:TI_RTE_S-PWQFN-N16" H 2250 1750 60  0001 C CNN
 F 3 "" H 2250 1750 60  0001 C CNN
+F 4 "TPS62095RGTR" H 2250 1550 50  0001 C CNN "MPN"
 	1    2250 1550
 	1    0    0    -1
@@
 F 2 "TI:TI_RTE_S-PWQFN-N16" H 7500 3950 60  0001 C CNN
 F 3 "" H 7500 3950 60  0001 C CNN
+F 4 "TPS62095RGTR" H 7500 3750 50  0001 C CNN "MPN"
 	1    7500 3750
 	1    0    0    -1
@@
 F 2 "Package_TO_SOT_SMD:SOT-23-5" H 5250 6075 50  0001 C CNN
 F 3 "http://www.diodes.com/_files/datasheets/AP131.pdf" H 5250 5750 50  0001 C CNN
+F 4 "AP131-25" H 5250 5750 50  0001 C CNN "MPN"
 	1    5250 5750
 	1    0    0    -1
@@
 F 2 "TI:TI_RTE_S-PWQFN-N16" H 7500 1750 60  0001 C CNN
 F 3 "" H 7500 1750 60  0001 C CNN
+F 4 "TPS62095RGTR" H 7500 1550 50  0001 C CNN "MPN"
 	1    7500 1550
 	1    0    0    -1
@@
 F 2 "TI:TI_RTE_S-PWQFN-N16" H 2250 4100 60  0001 C CNN
 F 3 "" H 2250 4100 60  0001 C CNN
+F 4 "TPS62095RGTR" H 2250 3900 50  0001 C CNN "MPN"
 	1    2250 3900
 	1    0    0    -1

Commit message: cleaning up MPN
Parts:
- L1, L3, L4: MPN (none) -> XAL4020-102ME; Part Number XAL4020-102ME -> (none)
- L2: MPN (none) -> XAL4020-102ME; Part Nunber XAL4020-102ME -> (none)

Commit message: Added in all the part numbers
Parts:
- C10, C11, C14, C15, C16, C17, C22, C23, C24, C25, C6, C9: MPN (none) -> CL21A226MQQNNNE
- C12, C18, C20, C7: MPN (none) -> CL05B103KB5NNNC
- C13, C8: MPN (none) -> CL05B471KB5NNNC
- C19, C21: MPN (none) -> CC0402KRX7R9BB562
- C26, C28: MPN (none) -> GRM21BR70J106KE76L
- C27: MPN (none) -> CC0402KRX7R7BB104
- R10: MPN (none) -> RTT021203FTH; Tolerance (none) -> 1%
- R11: MPN (none) -> RTT021103FTH; Tolerance (none) -> 1%
- R12: MPN (none) -> 0402WGF1603TCE; Tolerance (none) -> 1%
- R13: MPN (none) -> 0402WGF8202TCE; Tolerance (none) -> 1%
- R14: MPN (none) -> ERJPA2F2203X; Tolerance (none) -> 1%
- R15, R16, R17, R18, R19: MPN (none) -> RC0402JR-070RL
- R7: MPN (none) -> RTT024703FTH; Tolerance (none) -> 1%
- R8: MPN (none) -> RC0402FR-07150KL; Tolerance (none) -> 1%
- R9: MPN (none) -> RC0402FR-07330KL; Tolerance (none) -> 1%

Commit message: Part numbers are _properly_ in now.
Parts:
- R10, R11, R12, R13, R14, R7, R8, R9: Tolerance 1% -> (none)
